File: AW9523.brd (EAGLE design)
At the start: 27.9 x 22.9 mm, 15 parts, among them IC1 AW9523

Commit message: changed PWR label position, 2mm Via to GND
Parts:
- moved PWR 2.54 mm to (22.0, 14.8)
- moved R1 2.54 mm to (22.2, 12.7)
- moved R2 2.54 mm to (22.2, 16.8)
- moved R3 2.54 mm to (22.2, 7.62)
- moved R4 2.54 mm to (22.2, 10.2)
- moved C1 2.54 mm to (12.2, 15.5)
- moved IC1 2.54 mm to (15.2, 10.2)
- moved SV2 2.54 mm to (14.0, 2.54)
- moved SV3 2.54 mm to (14.0, 20.3)
- moved A0 2.54 mm to (6.51, 11.3)
- moved A1 2.54 mm to (6.51, 9.05)
- moved R5 2.54 mm to (6.51, 13.4)
- moved R6 2.54 mm to (6.51, 6.91)
- moved C2 2.54 mm to (14.3, 15.5)
- moved SV1 2.54 mm to (25.4, 11.4)
Routing:
- net GND: vias 90 -> 94
